File: src/DriveUnit_Bseries.kicad_pcb (KiCad board)
At the start: 2 copper layers, 65.7 x 51 mm, 56 parts, among them IC1 A3921, SW1 TVAF06-A020B-R, SW2 TVAF06-A020B-R, SW3 THAF01-NC-R, SW4 SS-12D00G3

Commit message: 基板デザインの完成
Parts:
- added G***: LOGO, 彼女(仮)_回路図:メカテック部ロゴ_縮小, B.Cu at (170.7, 118.1)
Other:
- board text added: "B series"
- board text added: "DriveUnit"
- board text added: "ver 1.0"
