File: src/DriveUnit_B-series(ver1.0).kicad_pcb (KiCad board)
At the start: 2 copper layers, 65.7 x 51 mm, 57 parts, among them IC1 A3921, SW1 TVAF06-A020B-R, SW2 TVAF06-A020B-R, SW3 THAF01-NC-R, SW4 SS-12D00G3

Commit message: 意図的なconflict
Parts:
- removed G***: LOGO, 彼女(仮)_回路図:メカテック部ロゴ_縮小
- removed G***: LOGO, 彼女(仮)_回路図:MD_QRCODE
- 3813-HA1, 3813-HB1, 3813-LA1, 3813-LB1: footprint 彼女(仮)_回路図:TO-220AB-NOHOLE -> DriveUnit_B-series(ver1.0):TO-220AB-NOHOLE
- C1, C2, C3, C4, C5, C7, C8: footprint 彼女(仮)_回路図:GCM188L81H104KA57 -> DriveUnit_B-series(ver1.0):GCM188L81H104KA57
- C10, C11: footprint 彼女(仮)_回路図:35PZJ330M10X9 -> DriveUnit_B-series(ver1.0):35PZJ330M10X9
- C12: footprint 彼女(仮)_回路図:GRM32ER7YA106KA12 -> DriveUnit_B-series(ver1.0):GRM32ER7YA106KA12
- C13: footprint 彼女(仮)_回路図:GRM21BC72A105KE01 -> DriveUnit_B-series(ver1.0):GRM21BC72A105KE01
- C6: footprint 彼女(仮)_回路図:GCM21BR71H474KA55 -> DriveUnit_B-series(ver1.0):GCM21BR71H474KA55
- C9: footprint 彼女(仮)_回路図:GRT31CC81H225KE01L -> DriveUnit_B-series(ver1.0):GRT31CC81H225KE01L
- D1, D8, D9: footprint 彼女(仮)_回路図:GS1010FL -> DriveUnit_B-series(ver1.0):GS1010FL
- EDGE1: footprint 彼女(仮)_回路図:10046971-019LF -> DriveUnit_B-series(ver1.0):10046971-019LF
- IC1: footprint 彼女(仮)_回路図:A3921 -> DriveUnit_B-series(ver1.0):A3921
- LED1, LED2, LED3, LED4, LED5: footprint 彼女(仮)_回路図:SML-E12V8WT86 -> DriveUnit_B-series(ver1.0):SML-E12V8WT86
- R1, R10, R11, R12, R13, R14, R15, R16, R18, R19, R2, R20, R21, R22, R3, R5, R6, R7, R8, R9: footprint 彼女(仮)_回路図:RG2012 -> DriveUnit_B-series(ver1.0):RG2012
- SW1, SW2: footprint 彼女(仮)_回路図:TVAF06-A020B-R -> DriveUnit_B-series(ver1.0):TVAF06-A020B-R
- SW3: footprint 彼女(仮)_回路図:THAF01-NC-R -> DriveUnit_B-series(ver1.0):THAF01-NC-R
- SW4: footprint 彼女(仮)_回路図:SS-12D00G3 -> DriveUnit_B-series(ver1.0):SS-12D00G3
- TLP1, TLP2: footprint 彼女(仮)_回路図:TLP2366 -> DriveUnit_B-series(ver1.0):TLP2366
- TR1, TR2: footprint 彼女(仮)_回路図:2SC3325 -> DriveUnit_B-series(ver1.0):2SC3325
- moved C11 0.73 mm to (161.8, 115.7)
Routing:
- net VCC: track 53.9 -> 49.6 mm
- net GND: track 82.4 -> 79.3 mm
- net /GLB: track 8.97 -> 6.35 mm, vias 0 -> 2
- net /SB: track 99.2 -> 97.0 mm
- net /GHB: track 15.5 -> 17.4 mm
- net /SA: track 59.3 -> 61.0 mm
- net /FF2: track 14.4 -> 15.0 mm
Other:
- board text removed: "B series"
- board text removed: "DriveUnit"
- board text removed: "FF1"
- board text removed: "FF2"
- board text removed: "LAP"
- board text removed: "POW"
- board text removed: "RESET"
- board text removed: "SA"
- board text removed: "SB"
- board text removed: "SM"
- board text removed: "Schematic"
- board text removed: "ver 1.0"
