File: src/DriveUnit_B-series(ver1.0).kicad_pcb (KiCad board)
At the start: 2 copper layers, 65.7 x 51 mm, 55 parts, among them IC1 A3921, SW1 TVAF06-A020B-R, SW2 TVAF06-A020B-R, SW3 THAF01-NC-R, SW4 SS-12D00G3

Commit message: conflict old側
Parts:
- added G***: LOGO, 彼女(仮)_回路図:メカテック部ロゴ_縮小, B.Cu at (170.7, 118.1)
- added G***: LOGO, 彼女(仮)_回路図:MD_QRCODE, B.Cu at (133.3, 90.2)
- 3813-HA1, 3813-HB1, 3813-LA1, 3813-LB1: footprint DriveUnit_B-series(ver1.0):TO-220AB-NOHOLE -> 彼女(仮)_回路図:TO-220AB-NOHOLE
- C1, C2, C3, C4, C5, C7, C8: footprint DriveUnit_B-series(ver1.0):GCM188L81H104KA57 -> 彼女(仮)_回路図:GCM188L81H104KA57
- C10, C11: footprint DriveUnit_B-series(ver1.0):35PZJ330M10X9 -> 彼女(仮)_回路図:35PZJ330M10X9
- C12: footprint DriveUnit_B-series(ver1.0):GRM32ER7YA106KA12 -> 彼女(仮)_回路図:GRM32ER7YA106KA12
- C13: footprint DriveUnit_B-series(ver1.0):GRM21BC72A105KE01 -> 彼女(仮)_回路図:GRM21BC72A105KE01
- C6: footprint DriveUnit_B-series(ver1.0):GCM21BR71H474KA55 -> 彼女(仮)_回路図:GCM21BR71H474KA55
- C9: footprint DriveUnit_B-series(ver1.0):GRT31CC81H225KE01L -> 彼女(仮)_回路図:GRT31CC81H225KE01L
- D1, D8, D9: footprint DriveUnit_B-series(ver1.0):GS1010FL -> 彼女(仮)_回路図:GS1010FL
- EDGE1: footprint DriveUnit_B-series(ver1.0):10046971-019LF -> 彼女(仮)_回路図:10046971-019LF
- IC1: footprint DriveUnit_B-series(ver1.0):A3921 -> 彼女(仮)_回路図:A3921
- LED1, LED2, LED3, LED4, LED5: footprint DriveUnit_B-series(ver1.0):SML-E12V8WT86 -> 彼女(仮)_回路図:SML-E12V8WT86
- R1, R10, R11, R12, R13, R14, R15, R16, R18, R19, R2, R20, R21, R22, R3, R5, R6, R7, R8, R9: footprint DriveUnit_B-series(ver1.0):RG2012 -> 彼女(仮)_回路図:RG2012
- SW1, SW2: footprint DriveUnit_B-series(ver1.0):TVAF06-A020B-R -> 彼女(仮)_回路図:TVAF06-A020B-R
- SW3: footprint DriveUnit_B-series(ver1.0):THAF01-NC-R -> 彼女(仮)_回路図:THAF01-NC-R
- SW4: footprint DriveUnit_B-series(ver1.0):SS-12D00G3 -> 彼女(仮)_回路図:SS-12D00G3
- TLP1, TLP2: footprint DriveUnit_B-series(ver1.0):TLP2366 -> 彼女(仮)_回路図:TLP2366
- TR1, TR2: footprint DriveUnit_B-series(ver1.0):2SC3325 -> 彼女(仮)_回路図:2SC3325
- moved C11 0.73 mm to (161.4, 116.3)
Routing:
- net VCC: track 49.6 -> 53.9 mm
- net GND: track 79.3 -> 82.4 mm
- net /GLB: track 6.35 -> 8.97 mm, vias 2 -> 0
- net /SB: track 97.0 -> 99.2 mm
- net /GHB: track 17.4 -> 15.5 mm
- net /SA: track 61.0 -> 59.3 mm
- net /FF2: track 15.0 -> 14.4 mm
Other:
- board text added: "B series"
- board text added: "DriveUnit"
- board text added: "FF1"
- board text added: "FF2"
- board text added: "LAP"
- board text added: "POW"
- board text added: "RESET"
- board text added: "SA"
- board text added: "SB"
- board text added: "SM"
- board text added: "Schematic"
- board text added: "ver 1.0"
