File: src/DriveUnit_B-series(ver1.0).brd (EAGLE design)
At the start: 65.7 x 51 mm, 55 parts, among them IC1 A3921, SW1 TVAF06-A020B-R, SW2 TVAF06-A020B-R, SW3 THAF01-NC-R, SW4 SS-12D00G3

Commit message: conflict前段階
Routing:
- net SB: track 97.0 -> 93.8 mm
- net VCC: track 49.6 -> 47.3 mm
- net GLB: track 6.35 -> 8.70 mm, vias 2 -> 0
- net SA: track 61.0 -> 59.0 mm
- net GHB: track 17.4 -> 15.5 mm
- net FF2: track 15.0 -> 14.4 mm
