File: src/(KiCad)DriveUnit_B-series(ver2.0).kicad_pcb (KiCad board)
At the start: 2 copper layers, 65.7 x 51 mm, 67 parts, among them SW3 THAF01-NC-R, SW4 SS-12D00G3

Commit message: デザイン完了
Parts:
- added G***: LOGO, (Eagle)DriveUnit_B-series(ver2.0):メカテック部ロゴ_縮小, B.Cu at (126.1, 117.5)
- added G***: LOGO, (Eagle)DriveUnit_B-series(ver2.0):MD_QRCODE(large2), B.Cu at (132.5, 87.9)
- renumbered R14 to R14]
Other:
- board text added: "Copyright © 2022 Issaimaru All Rights Reserved."
- board text added: "D1"
- board text added: "D2"
- board text added: "D3"
- board text added: "D4"
- board text added: "D5"
- board text added: "D6"
- board text added: "R14"
- board text added: "R2"
- board text added: "R26"
- board text added: "R27"
- board text added: "document"
- board text added: "ver 2.0"

Commit message: ver2.0完全完了_gerber出力前
Parts:
- moved C11 7.31 mm to (152.9, 116.5), turned to 90 degrees
- moved C13 4.41 mm to (148.0, 112.3)
- moved C12 3.21 mm to (150.5, 111.8)
- moved TR1 0.30 mm to (174.9, 92.1)
- moved TR2 0.30 mm to (179.2, 92.1)
- moved R4 0.25 mm to (172.7, 94.2)
- moved R5 0.25 mm to (179.6, 94.2)
- moved R25 0.12 mm to (175.2, 93.5)
Routing:
- net GND: track 61.3 -> 53.8 mm
- net Net-(D5-PadC): track 11.1 -> 8.83 mm
- net /LAP: track 20.1 -> 21.3 mm
- net /V5: track 59.9 -> 61.0 mm
- net VCC: vias 11 -> 8
