File: src/(KiCad)DriveUnit_B-series(ver2.0).kicad_pcb (KiCad board)
At the start: 2 copper layers, 65.7 x 51 mm, 65 parts, among them IC1 A3921, SW1 TVAF06-A020B-R, SW2 TVAF06-A020B-R, SW3 THAF01-NC-R, SW4 SS-12D00G3

Commit message: 表デザイン完成
Parts:
- moved R11 2.05 mm to (174.1, 113.0)
- moved TR1 0.30 mm to (174.9, 92.1)
- moved TR2 0.30 mm to (179.2, 92.1)
- renumbered HA1 to HA, HB1 to HB, LA1 to LA, LB1 to LB, SW3 to RESET, SW1 to SA, SW2 to SB
Routing:
- net GND: track 56.8 -> 59.1 mm
- net /RESET: track 48.7 -> 49.2 mm
Other:
- board text added: "B series"
- board text added: "D4"
- board text added: "D5"
- board text added: "DriveUnit"
- board text added: "LAP"
- board text added: "SM"

Commit message: デザイン途中まで
Parts:
- moved TR3 1.14 mm to (177.1, 94.0)
- moved TR4 1.14 mm to (173.0, 94.0)
- moved R21 0.75 mm to (156.9, 102.5)
- moved R14 0.73 mm to (169.7, 81.2)
- moved R12 0.70 mm to (164.9, 100.2)
- moved R20 0.70 mm to (156.9, 100.2)
- moved C9 0.68 mm to (163.8, 98.0)
- moved R13 0.64 mm to (166.9, 83.8)
- moved R10 0.60 mm to (164.9, 102.5)
- moved C4 0.39 mm to (163.0, 96.0)
- renumbered IC1 to A3921
Routing:
- net /V5: track 57.9 -> 52.8 mm, vias 4 -> 2
- net /PWM: track 28.0 -> 31.1 mm
- net /SA: track 101.5 -> 104.1 mm
- net /DIR: track 46.8 -> 48.1 mm
- net Net-(IC1-Pad28): track 5.42 -> 6.60 mm
- net /LAP: track 25.2 -> 26.4 mm
- net Net-(D2-PadA): track 13.9 -> 15.0 mm
- net /SB: track 62.7 -> 63.7 mm
- net /GHA: track 10.3 -> 11.4 mm
- net GND: track 59.1 -> 58.2 mm
- net Net-(HA1-PadGATE): track 45.8 -> 46.6 mm
- net Net-(C4-PadP$2): track 5.02 -> 5.80 mm
- net /GHB: track 7.42 -> 8.19 mm
- net Net-(IC1-Pad27): track 2.15 -> 2.81 mm
- net /RESET: track 49.2 -> 49.8 mm
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Other:
- board text added: "D2"
- board text added: "D3"

Commit message: 基板デザインの完全完成_gerber出力前
Parts:
- added G***: LOGO, (Eagle)DriveUnit_B-series(ver2.0):メカテック部ロゴ_縮小, B.Cu at (126.1, 117.5)
- added G***: LOGO, (Eagle)DriveUnit_B-series(ver2.0):MD_QRCODE(large2), B.Cu at (132.5, 87.9)
Routing:
- net Net-(HA1-PadGATE): track 46.6 -> 45.5 mm
Other:
- board text added: "Copyright © 2022 Issaimaru All Rights Reserved."
- board text added: "D1"
- board text added: "document"
- board text added: "ver 2.0"
